File: power_control.sch (KiCad schematic (older format))
At the start: 80 parts, among them J26 Conn_01x02, J27 Conn_01x02, J28 Conn_01x02, J29 Conn_01x02, J30 Conn_01x02, J31 Conn_01x02, J32 Conn_01x02, J33 Conn_01x02, U10 L6203, U11 L6203, U12 L6203, U5 L6203, U6 L6203, U7 L6203, U8 L6203, U9 L6203

Commit message: Removed L6203
Parts:
- removed C11, C12, C13, C14, C31, C32, C33, C34: 220nF, lsts-passives:C_0603, symbol Device:C
- removed C15, C18, C21, C24, C35, C38, C41, C44: 100nF, lsts-passives:C_0603, symbol Device:C
- removed C16, C17, C19, C20, C22, C23, C25, C26, C36, C37, C39, C40, C42, C43, C45, C46: 15nF, lsts-passives:C_0603, symbol Device:C
- removed C27, C28, C29, C30, C47, C48, C49, C50: 22nF, lsts-passives:C_0603, symbol Device:C
- removed D10, D11, D12, D13, D14, D15, D16, D17, D18, D19, D20, D21, D22, D23, D24, D9: SDT5100LP5-13, Diode_SMD:D_PowerDI-5, symbol Device:D
- removed J26, J27, J28, J29, J30, J31, J32, J33: Conn_01x02, Connector_Molex:Molex_Micro-Fit_3.0_43045-0212_2x01_P3.00mm_Vertical, symbol Connector_Generic:Conn_01x02
- removed R30, R31, R32, R33, R34, R35, R36, R37: 10R, lsts-passives:R_0603, symbol Device:R
- removed U10, U11, U12, U5, U6, U7, U8, U9: L6203, lsts-discretes:MULTIWATT-11, symbol lsts-devices:L6203
Connections:
- net labels removed: +12V, GND, MTR1_BW, MTR1_EN, MTR1_FW, MTR2_BW, MTR2_EN, MTR2_FW, MTR3_BW, MTR3_EN, MTR3_FW, MTR4_BW, MTR4_EN, MTR4_FW, MTR5_BW, MTR5_EN, MTR5_FW, MTR6_BW, MTR6_EN, MTR6_FW, MTR7_BW, MTR7_EN, MTR7_FW, MTR8_BW, MTR8_EN, MTR8_FW
- wire segments 280 -> 0

Commit message: Added DRV8801PWP to schematic
Parts:
- added C11, C12, C13, C14, C15, C16, C18, C20, C22, C23, C24, C25, C26, C27, C28, C30, C32, C34, C35, C36, C37, C38, C40, C42: 100nF, lsts-passives:C_0603, symbol Device:C
- added C17, C19, C21, C29, C31, C33, C39, C41: 100uF, Capacitor_THT:CP_Radial_D5.0mm_P2.00mm, symbol Device:CP
- added J26, J27, J28, J29, J30, J31, J32, J33: Conn_01x02, Connector_Molex:Molex_Micro-Fit_3.0_43045-0212_2x01_P3.00mm_Vertical, symbol Connector_Generic:Conn_01x02
- added R30, R31, R32, R33, R34, R35, R36, R37, R38, R39, R40, R41, R42, R43, R44, R45: 10kR, lsts-passives:R_0603, symbol Device:R
- added U10, U11, U12, U5, U6, U7, U8, U9: DRV8801PWP, Package_SO:HTSSOP-16-1EP_4.4x5mm_P0.65mm_EP3.4x5mm_Mask3x3mm_ThermalVias, symbol Driver_Motor:DRV8801PWP
Connections:
- net labels added: +12V, +5V, GND, MTR1_EN, MTR1_PH, MTR1_SL, MTR2_EN, MTR2_PH, MTR2_SL, MTR3_EN, MTR3_PH, MTR3_SL, MTR4_EN, MTR4_PH, MTR4_SL, MTR5_EN, MTR5_PH, MTR5_SL, MTR6_EN, MTR6_PH, MTR6_SL, MTR7_EN, MTR7_PH, MTR7_SL, MTR8_EN, MTR8_PH, MTR8_SL
- wire segments 0 -> 224
- no-connect marks 0 -> 16
