File: power_passive.sch (KiCad schematic (older format))
At the start: 39 parts, among them J10 Conn_01x02, J11 Conn_01x02, J12 Conn_01x02, J13 Conn_01x02, J14 Conn_01x02, J15 Conn_01x02, J16 Conn_01x02, J17 Conn_01x02, J18 Conn_01x02, J19 Conn_01x02, J20 Conn_01x02, J5 ATX-24, J6 Conn_01x02, J7 Conn_01x02, J8 Conn_01x02, J9 Conn_01x02, Q1 MMBT4401-7-F, Q10 MMBT4401-7-F, Q11 SI7113ADN-T1-GE3, Q2 MMBT4401-7-F, Q3 MMBT4401-7-F, Q4 SI7113ADN-T1-GE3, Q5 SI7113ADN-T1-GE3, Q6 MMBT4401-7-F, Q7 MMBT4401-7-F, Q8 SI7113ADN-T1-GE3, Q9 SI7113ADN-T1-GE3

Commit message: Final touches
Parts:
- Q1, Q10, Q2, Q3, Q6, Q7: footprint lsts-discretes:SOT23_BC817 -> lsts_discretes:SOT23_BC817
- Q11, Q4, Q5, Q8, Q9: footprint lsts-discretes:PowerPAK_1212-8 -> lsts_discretes:PowerPAK_1212-8
- R10, R11, R12, R13, R14, R15, R16, R17, R18, R19, R8, R9: footprint lsts-passives:R_0603 -> lsts_passives:R_0603
- renumbered J11 to J10, J12 to J11, J13 to J12, J14 to J13, J15 to J14, J16 to J15, J17 to J16, J18 to J17, J19 to J18, J20 to J19, J5 to J4, J6 to J5, J7 to J6, J8 to J7, J9 to J8, J10 to J9

Commit message: Small fix
Parts:
- removed R9: 10kR, lsts_passives:R_0603, symbol Device:R
Changed lines of the file:
@@
 Wire Wire Line
 	8600 5450 8600 5950
-Wire Wire Line
-	2500 1450 2600 1450
 Text HLabel 2200 1350 1    50   Input ~ 0
 PWR_CTR
@@
 	1    0    0    -1
 $EndComp
-$Comp
-L Device:R R?
-U 1 1 5E39FAB3
-P 2600 1300
-AR Path="/5E39FAB3" Ref="R?"  Part="1"
-AR Path="/5E1C04CF/5E39FAB3" Ref="R?"  Part="1"
-AR Path="/5E3E0C4B/5E39FAB3" Ref="R?"  Part="1"
-AR Path="/5E4850C0/5E39FAB3" Ref="R?"  Part="1"
-AR Path="/5E4060AB/5E39FAB3" Ref="R9"  Part="1"
-F 0 "R9" V 2393 1300 50  0000 C CNN
-F 1 "10kR" V 2484 1300 50  0000 C CNN
-F 2 "lsts_passives:R_0603" V 2530 1300 50  0001 C CNN
-F 3 "~" H 2600 1300 50  0001 C CNN
-F 4 "CRCW060310K0JNEBC" H 2600 1300 50  0001 C CNN "manf#"
-	1    2600 1300
-	1    0    0    -1
-$EndComp
-Connection ~ 2600 1450
-Wire Wire Line
-	2600 1450 2750 1450
-Text HLabel 2600 1150 1    50   Input ~ 0
-+5V_SB
 Wire Wire Line
 	8150 2000 8000 2000
@@
 	0    -1   -1   0
 $EndComp
+Wire Wire Line
+	2500 1450 2750 1450
 $EndSCHEMATC
